File: motor_controller_encoder_counter.kicad_pcb (KiCad board)
At the start: 4 copper layers, 30 x 40 mm, 24 parts, among them J1 Conn_01x04_Pin, J2 JST, J3 WAGO_2pos_3.5mm_Horizontal, J4 Motor Driver Power, J6 Motor Driver Logic, J8 JST, U1 LS7866C, U2 LS7866C

Commit message: ready for review
Parts:
- added G***: LOGO, HPRC_Graphics:ncsu_logo, B.Cu at (28.9, 47.8)
- added R5: 2.2k, Resistor_SMD:R_0402_1005Metric, F.Cu at (35.7, 47.5)
- added R6: 2.2k, Resistor_SMD:R_0402_1005Metric, F.Cu at (24.8, 45.8)
- C1, C2, C3, C5, C6, C7: footprint Capacitor_SMD:C_0603_1608Metric -> Capacitor_SMD:C_0402_1005Metric
- C4: value 47u -> 100u
- R1, R2, R3, R4: footprint Resistor_SMD:R_0603_1608Metric -> Resistor_SMD:R_0402_1005Metric
- moved R1 2.17 mm to (25.5, 24.9), turned to 180 degrees
- moved G*** 2.00 mm to (23.1, 50.5)
- moved C1 1.41 mm to (28.8, 24.4), turned to 0 degrees
- moved C5 1.35 mm to (30.1, 31.5), turned to -90 degrees
- moved R2 1.10 mm to (27.1, 24.0), turned to -90 degrees
Connections:
- net +5V renamed +3.3V
Routing:
- net +3.3V: track 20.9 -> 26.4 mm, vias 5 -> 8
- net GND: track 28.5 -> 30.0 mm
- net Net-(U1-A2): track 4.89 -> 3.51 mm
- net /SCL: track 56.5 -> 57.1 mm
- net /SDA: track 53.8 -> 53.9 mm, vias 3 -> 4
Other:
- board text added: "+3.3V"
- board text removed: "+5V"
