File: motor_controller_encoder_counter.kicad_pcb (KiCad board)
At the start: 4 copper layers, 30 x 40 mm, 27 parts, among them J1 Conn_01x04_Pin, J2 JST, J3 WAGO_2pos_3.5mm_Horizontal, J4 Motor Driver Power, J6 Motor Driver Logic, J8 JST, U1 LS7866C, U2 LS7866C

Commit message: ready to review
Parts:
- moved TP4 0.41 mm to (25.8, 32.2)
Routing:
- net Net-(U1-DFLAG/): track 0.48 -> 3.77 mm
- net Net-(U2-A2): track 3.85 -> 4.89 mm
- net /SCL: track 57.1 -> 56.4 mm
- net /SDA: track 53.9 -> 54.4 mm
- net +3.3V: track 26.4 -> 26.1 mm, vias 8 -> 7
Other:
- outline, holes or cut-outs redrawn

Commit message: ordered
Parts:
- added H1: MountingHole, MountingHole:MountingHole_2.2mm_M2, F.Cu at (22.5, 18.0)
- added H2: MountingHole, MountingHole:MountingHole_2.2mm_M2, F.Cu at (47.5, 18.0)
- added H3: MountingHole, MountingHole:MountingHole_2.2mm_M2, F.Cu at (47.5, 62.5)
- added H4: MountingHole, MountingHole:MountingHole_2.2mm_M2, F.Cu at (22.5, 62.5)
Other:
- board size 30 x 40 mm -> 30 x 49.5 mm
