File: motor_controller_encoder_counter.kicad_sch (KiCad schematic)
At the start: 7 parts, among them J1 Conn_01x04_Pin, J3 WAGO_2pos_3.5mm_Horizontal, J4 Motor Driver Power, J6 Motor Driver Logic

Commit message: ready for review
Parts:
- added R5, R6: 2.2k, Resistor_SMD:R_0402_1005Metric, symbol Device:R_Small
- C2, C7: footprint Capacitor_SMD:C_0603_1608Metric -> Capacitor_SMD:C_0402_1005Metric
- C4: value 47u -> 100u
- J1, J4, J6: now not fitted; now left out of the parts list
Connections:
- net SCL: now also R6.2
- net SDA: now also R5.2
- net +5V renamed +3.3V
- net +3.3V: now also R5.1, R6.1

Commit message: ordered
Parts:
- added H1, H2, H3, H4: MountingHole, MountingHole:MountingHole_2.2mm_M2, symbol Mechanical:MountingHole
- C2, C7: Manufacturer Name (none) -> Murata Electronics; Manufacturer PN (none) -> GRM155R61C225KE44D
- C4: Manufacturer Name (none) -> Chemi-Con; Manufacturer PN (none) -> APXG160ARA101ME61G
- J3: Manufacturer Name (none) -> WAGO Corporation; Manufacturer PN (none) -> 2601-1102
- R5, R6: Manufacturer Name (none) -> YAGEO; Manufacturer PN (none) -> RC0402FR-072k2L
